File: hw/Grid64_v3/Grid64_v3.kicad_sch (KiCad schematic)
At the start: 220 parts, among them J3 Btn_Row, J4 Btn_Col, U1 XIAO-ESP32-C3-DIP, U2 74LVC2T45DC, U3 74LVC2T45DC

Commit message: Fixing the firmware and the hardware
Parts:
- L1: footprint Switch_Misc:MX-LED-PolarityMarked -> Switch_Misc:MX-LED
Connections:
- net GND: now also PISO1.10 (DS)
- net PISO_DATA: now also PISO1.9 (Q7); no longer PISO1.10 (DS)
- no-connect marks 7 -> 6
Other:
- moved on the sheet: C3
Changed lines of the file:
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@@
 	)
 	(no_connect
-		(at 261.62 173.99)
-	)
-	(no_connect
 		(at 360.68 198.12)
 	)
@@
 	(wire
 		(pts
+			(xy 222.25 173.99) (xy 236.22 173.99)
+		)
+		(stroke
+			(width 0)
+			(type default)
+		)
+	)
+	(wire
+		(pts
 			(xy 54.61 179.07) (xy 67.31 179.07)
 		)
@@
 	(wire
 		(pts
-			(xy 267.97 172.72) (xy 267.97 171.45)
+			(xy 278.13 172.72) (xy 278.13 171.45)
 		)
 		(stroke
@@
 	(wire
 		(pts
-			(xy 267.97 163.83) (xy 248.92 163.83)
+			(xy 278.13 163.83) (xy 248.92 163.83)
 		)
 		(stroke
@@
 	(wire
 		(pts
-			(xy 267.97 163.83) (xy 267.97 167.64)
+			(xy 278.13 163.83) (xy 278.13 167.64)
 		)
 		(stroke
@@
 	(wire
 		(pts
+			(xy 222.25 177.8) (xy 222.25 173.99)
+		)
+		(stroke
+			(width 0)
+			(type default)
+		)
+	)
+	(wire
+		(pts
 			(xy 363.22 124.46) (xy 363.22 127)
 		)
@@
 	(global_label "PISO_DATA"
 		(shape input)
-		(at 236.22 173.99 180)
+		(at 261.62 173.99 0)
 		(fields_autoplaced yes)
 		(effects
@@
 				(size 1.27 1.27)
 			)
-			(justify right)
+			(justify left)
 		)
 		(property "Intersheetrefs" "${INTERSHEET_REFS}"
-			(at 223.4376 173.99 0)
+			(at 274.4024 173.99 0)
 			(effects
 				(font
 					(size 1.27 1.27)
 				)
-				(justify right)
+				(justify left)
 				(hide yes)
 			)
@@
 	(symbol
 		(lib_id "power:GND")
-		(at 267.97 171.45 0)
+		(at 278.13 171.45 0)
 		(unit 1)
 		(exclude_from_sim no)
@@
 		(fields_autoplaced yes)
 		(property "Reference" "#PWR018"
-			(at 267.97 177.8 0)
+			(at 278.13 177.8 0)
 			(effects
 				(font
@@
 		)
 		(property "Value" "GND"
-			(at 267.97 176.53 0)
+			(at 278.13 176.53 0)
 			(effects
 				(font
@@
 		)
 		(property "Footprint" ""
-			(at 267.97 171.45 0)
+			(at 278.13 171.45 0)
 			(effects
 				(font
@@
 		)
 		(property "Datasheet" ""
-			(at 267.97 171.45 0)
+			(at 278.13 171.45 0)
 			(effects
 				(font
@@
 		)
 		(property "Description" "Power symbol creates a global label with name \"GND\" , ground"
-			(at 267.97 171.45 0)
+			(at 278.13 171.45 0)
 			(effects
 				(font
@@
 			)
 		)
-		(property "Footprint" "Switch_Misc:MX-LED-PolarityMarked"
+		(property "Footprint" "Switch_Misc:MX-LED"
 			(at 283.21 60.96 0)
 			(effects
@@
 	)
 	(symbol
+		(lib_id "power:GND")
+		(at 222.25 177.8 0)
+		(unit 1)
+		(exclude_from_sim no)
+		(in_bom yes)
+		(on_board yes)
+		(dnp no)
+		(fields_autoplaced yes)
+		(property "Reference" "#PWR032"
+			(at 222.25 184.15 0)
+			(effects
+				(font
+					(size 1.27 1.27)
+				)
+				(hide yes)
+			)
+		)
+		(property "Value" "GND"
+			(at 222.25 182.88 0)
+			(effects
+				(font
+					(size 1.27 1.27)
+				)
+			)
+		)
+		(property "Footprint" ""
+			(at 222.25 177.8 0)
+			(effects
+				(font
+					(size 1.27 1.27)
+				)
+				(hide yes)
+			)
+		)
+		(property "Datasheet" ""
+			(at 222.25 177.8 0)
+			(effects
+				(font
+					(size 1.27 1.27)
+				)
+				(hide yes)
+			)
+		)
+		(property "Description" "Power symbol creates a global label with name \"GND\" , ground"
+			(at 222.25 177.8 0)
+			(effects
+				(font
+					(size 1.27 1.27)
+				)
+				(hide yes)
+			)
+		)
+		(pin "1"
+		)
+		(instances
+			(project "Grid64_v3"
+				(path "/b952a6af-3a15-4f89-b286-823bbef71c7d"
+					(reference "#PWR032")
+					(unit 1)
+				)
+			)
+		)
+	)
+	(symbol
 		(lib_id "ScottoKeebs:Placeholder_Keyswitch")
 		(at 77.47 67.31 0)
@@
 	(symbol
 		(lib_id "Device:C_Small")
-		(at 267.97 170.18 0)
+		(at 278.13 170.18 0)
 		(unit 1)
 		(exclude_from_sim no)
@@
 		(dnp no)
 		(property "Reference" "C3"
-			(at 265.68 168.93 90)
+			(at 275.84 168.93 90)
 			(effects
 				(font
@@
 		)
 		(property "Value" "0.1uF"
-			(at 270.27 168.93 90)
+			(at 280.43 168.93 90)
 			(effects
 				(font
@@
 		)
 		(property "Footprint" "Capacitor_SMD:C_0805_2012Metric"
-			(at 267.97 170.18 0)
+			(at 278.13 170.18 0)
 			(effects
 				(font
@@
 		)
 		(property "Datasheet" "~"
-			(at 267.97 170.18 0)
+			(at 278.13 170.18 0)
 			(effects
 				(font
@@
 		)
 		(property "Description" "Unpolarized capacitor, small symbol"
-			(at 267.97 170.18 0)
+			(at 278.13 170.18 0)
 			(effects
 				(font
@@
 		)
 		(property "LCSC" "C49678"
-			(at 267.97 170.18 90)
+			(at 278.13 170.18 90)
 			(effects
 				(font
