File: hw/Grid64_v3/Grid64_v3.kicad_pcb (KiCad board)
At the start: 2 copper layers, 157.2 x 176.2 mm, 229 parts, among them J3 Btn_Row, J4 Btn_Col, U1 XIAO-ESP32-C3-DIP, U2 74LVC2T45DC, U3 74LVC2T45DC

Commit message: Fixing the firmware and the hardware
Parts:
- D1, D10, D11, D12, D13, D14, D15, D16, D17, D18, D19, D2, D20, D21, D22, D23, D24, D25, D26, D27, D28, D29, D3, D30, D31, D32, D33, D34, D35, D36, D37, D38, D39, D4, D40, D41, D42, D43, D44, D45, D46, D47, D48, D49, D5, D50, D51, D52, D53, D54, D55, D56, D57, D58, D59, D6, D60, D61, D62, D63, D64, D7, D8, D9: value Diode -> 1N4148W
- L1: footprint Switch_Misc:MX-LED-PolarityMarked -> Switch_Misc:MX-LED
Connections:
- PISO1 pad 10: PISO_DATA -> GND
- PISO1 pad 9: unconnected-(PISO1-Q7-Pad9) -> PISO_DATA

Commit message: Lots of firmware improvements
Parts:
- moved C3 0.50 mm to (135.4, 38.6)
Routing:
- net GND: track 6.35 -> 5.25 mm, vias 45 -> 46
- net Row2: track 227.5 -> 228.3 mm
- net Row3: track 248.0 -> 248.6 mm
- net Row1: track 206.6 -> 207.2 mm
- net Row0: track 185.2 -> 185.7 mm
Other:
- board text added: "3.0 - JUL 2025 - Initial Design 3.1 - JUL 2025 - Fixed PISO pin assignments."
- board text removed: "3.0 - JUL 2025 - Initial Design"
